File: esp8266_breakout.kicad_pcb (KiCad board)
At the start: 2 copper layers, 42.5 x 45.1 mm, 46 parts, among them CON1 USB-MICRO-B2, P1 CONN_12, P2 CONN_2, Q1 MOS_P, Q2 MOS_N, SW1 SW_PUSH, U1 NCP1117LP, U2 ESP8266-3, U3 FT230XS

Commit message: Fixed footprints
Parts:
- FB1: footprint SM0603_Resistor -> SM0805
- moved G*** 7.85 mm to (80.0, 92.1)
- moved FB1 0.63 mm to (71.1, 89.5)
Routing:
- net VDD: track 7.61 -> 8.48 mm
Changed lines of the file:
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@@
     (thickness 1.6)
     (drawings 22)
-    (tracks 293)
+    (tracks 300)
     (zones 0)
     (modules 46)
@@
   (layers
     (15 F.Cu signal hide)
-    (0 B.Cu signal)
+    (0 B.Cu signal hide)
     (16 B.Adhes user)
     (17 F.Adhes user)
@@
   )
   (setup
-    (last_trace_width 0.2)
+    (last_trace_width 0.4)
     (user_trace_width 0.3)
     (user_trace_width 0.4)
@@
   )
   (module SM0603_Resistor (layer F.Cu)
-    (at 71.755 89.535 180)
-    (attr smd)
-    (fp_text reference FB1 (at 2.54 0 180) (layer F.SilkS)
-      (effects (font (size 0.75 0.75) (thickness 0.2)))
-    )
-    (fp_text value FILTER (at -1.69926 0 270) (layer F.SilkS)
-      (effects (font (size 0.508 0.4572) (thickness 0.1143)))
-    )
-    (fp_line (start -0.50038 -0.6985) (end -1.2065 -0.6985) (layer F.SilkS) (width 0.127))
-    (fp_line (start -1.2065 -0.6985) (end -1.2065 0.6985) (layer F.SilkS) (width 0.127))
-    (fp_line (start -1.2065 0.6985) (end -0.50038 0.6985) (layer F.SilkS) (width 0.127))
-    (fp_line (start 1.2065 -0.6985) (end 0.50038 -0.6985) (layer F.SilkS) (width 0.127))
-    (fp_line (start 1.2065 -0.6985) (end 1.2065 0.6985) (layer F.SilkS) (width 0.127))
-    (fp_line (start 1.2065 0.6985) (end 0.50038 0.6985) (layer F.SilkS) (width 0.127))
-    (pad 1 smd rect (at -0.762 0 180) (size 0.635 1.143)
-      (layers F.Cu F.Paste F.Mask)
-      (net 38 VDD)
-    )
-    (pad 2 smd rect (at 0.762 0 180) (size 0.635 1.143)
-      (layers F.Cu F.Paste F.Mask)
-      (net 37 VCC)
-    )
-    (model smd\resistors\R0603.wrl
-      (at (xyz 0 0 0.001))
-      (scale (xyz 0.5 0.5 0.5))
-      (rotate (xyz 0 0 0))
-    )
-  )
-  (module SM0603_Resistor (layer F.Cu)
     (at 90.17 92.71 90)
     (attr smd)
@@
   )
   (module chaosinkl_silkbot_25_00mm (layer B.Cu)
-    (at 72.39 90.17)
+    (at 80.01 92.075)
     (fp_text reference G*** (at 0 -9.3091) (layer B.SilkS) hide
       (effects (font (size 0.49784 0.49784) (thickness 0.09906)) (justify mirror))
@@
       (xy -0.21336 -4.14274) (xy -0.2159 -4.13004) (xy -0.2159 -4.10972) (xy -0.2159 -4.10972)) (layer B.SilkS) (width 0.00254))
   )
+  (module SM0805 (layer F.Cu)
+    (at 71.12 89.535 180)
+    (attr smd)
+    (fp_text reference FB1 (at 0 -0.3175 180) (layer F.SilkS)
+      (effects (font (size 0.50038 0.50038) (thickness 0.10922)))
+    )
+    (fp_text value FILTER (at 0 0.381 180) (layer F.SilkS)
+      (effects (font (size 0.50038 0.50038) (thickness 0.10922)))
+    )
+    (fp_circle (center -1.651 0.762) (end -1.651 0.635) (layer F.SilkS) (width 0.09906))
+    (fp_line (start -0.508 0.762) (end -1.524 0.762) (layer F.SilkS) (width 0.09906))
+    (fp_line (start -1.524 0.762) (end -1.524 -0.762) (layer F.SilkS) (width 0.09906))
+    (fp_line (start -1.524 -0.762) (end -0.508 -0.762) (layer F.SilkS) (width 0.09906))
+    (fp_line (start 0.508 -0.762) (end 1.524 -0.762) (layer F.SilkS) (width 0.09906))
+    (fp_line (start 1.524 -0.762) (end 1.524 0.762) (layer F.SilkS) (width 0.09906))
+    (fp_line (start 1.524 0.762) (end 0.508 0.762) (layer F.SilkS) (width 0.09906))
+    (pad 1 smd rect (at -0.9525 0 180) (size 0.889 1.397)
+      (layers F.Cu F.Paste F.Mask)
+      (net 38 VDD)
+    )
+    (pad 2 smd rect (at 0.9525 0 180) (size 0.889 1.397)
+      (layers F.Cu F.Paste F.Mask)
+      (net 37 VCC)
+    )
+    (model smd/chip_cms.wrl
+      (at (xyz 0 0 0))
+      (scale (xyz 0.1 0.1 0.1))
+      (rotate (xyz 0 0 0))
+    )
+  )
   (gr_text V.1.0 (at 62.23 77.47) (layer B.SilkS)
     (effects (font (size 0.9 0.9) (thickness 0.225)) (justify mirror))
@@
   (segment (start 87.884 87.884) (end 87.884 89.705) (width 0.4) (layer F.Cu) (net 36))
   (segment (start 87.63 87.63) (end 87.884 87.884) (width 0.4) (layer F.Cu) (net 36))
+  (via (at 68.58 89.535) (size 0.7) (layers F.Cu B.Cu) (net 37))
+  (segment (start 68.58 89.535) (end 68.58 81.915) (width 0.4) (layer B.Cu) (net 37))
+  (segment (start 71.882 81.407) (end 71.882 82.55) (width 0.4) (layer F.Cu) (net 37))
+  (segment (start 71.882 81.407) (end 71.12 80.645) (width 0.4) (layer F.Cu) (net 37))
+  (segment (start 71.12 80.645) (end 69.215 80.645) (width 0.4) (layer F.Cu) (net 37))
+  (via (at 69.215 80.645) (size 0.6) (drill 0.2) (layers F.Cu B.Cu) (net 37))
+  (segment (start 68.58 81.28) (end 69.215 80.645) (width 0.4) (layer B.Cu) (net 37))
+  (segment (start 68.58 81.915) (end 68.58 81.28) (width 0.4) (layer B.Cu) (net 37))
+  (segment (start 70.1675 89.535) (end 68.58 89.535) (width 0.4) (layer F.Cu) (net 37))
+  (segment (start 68.326 89.789) (end 68.58 89.535) (width 0.4) (layer F.Cu) (net 37))
+  (segment (start 68.326 89.789) (end 67.31 89.789) (width 0.4) (layer F.Cu) (net 37))
   (segment (start 95.885 67.31) (end 95.885 69.85) (width 0.4) (layer B.Cu) (net 37))
   (segment (start 93.98 89.535) (end 93.98 67.945) (width 0.4) (layer B.Cu) (net 37))
   (segment (start 93.345 90.17) (end 93.98 89.535) (width 0.4) (layer B.Cu) (net 37))
   (segment (start 92.075 90.17) (end 91.44 89.535) (width 0.4) (layer B.Cu) (net 37))
-  (segment (start 69.215 89.535) (end 81.915 89.535) (width 0.4) (layer B.Cu) (net 37))
+  (segment (start 68.58 89.535) (end 81.915 89.535) (width 0.4) (layer B.Cu) (net 37))
   (segment (start 91.44 89.535) (end 81.915 89.535) (width 0.4) (layer B.Cu) (net 37))
   (segment (start 92.075 90.17) (end 93.345 90.17) (width 0.4) (layer B.Cu) (net 37))
   (segment (start 94.615 67.31) (end 95.885 67.31) (width 0.4) (layer B.Cu) (net 37))
   (segment (start 93.98 67.945) (end 94.615 67.31) (width 0.4) (layer B.Cu) (net 37))
-  (segment (start 69.215 80.645) (end 69.215 89.535) (width 0.4) (layer B.Cu) (net 37))
-  (via (at 69.215 80.645) (size 0.6) (drill 0.2) (layers F.Cu B.Cu) (net 37))
-  (segment (start 71.12 80.645) (end 69.215 80.645) (width 0.4) (layer F.Cu) (net 37))
-  (via (at 69.215 89.535) (size 0.6) (drill 0.2) (layers F.Cu B.Cu) (net 37))
-  (segment (start 68.961 89.789) (end 69.215 89.535) (width 0.4) (layer F.Cu) (net 37))
-  (segment (start 71.882 81.407) (end 71.12 80.645) (width 0.4) (layer F.Cu) (net 37))
-  (segment (start 71.882 82.55) (end 71.882 81.407) (width 0.4) (layer F.Cu) (net 37))
   (segment (start 65.7225 87.122) (end 65.7225 89.7255) (width 0.4) (layer F.Cu) (net 37))
   (segment (start 65.7225 89.7255) (end 65.659 89.789) (width 0.4) (layer F.Cu) (net 37))
@@
   (segment (start 73.3425 84.7725) (end 73.152 84.582) (width 0.4) (layer F.Cu) (net 37))
   (segment (start 73.3425 84.7725) (end 74.803 84.7725) (width 0.4) (layer F.Cu) (net 37))
-  (segment (start 67.437 89.789) (end 65.659 89.789) (width 0.4) (layer F.Cu) (net 37))
-  (segment (start 67.437 89.789) (end 68.961 89.789) (width 0.4) (layer F.Cu) (net 37))
-  (segment (start 69.215 89.535) (end 70.993 89.535) (width 0.4) (layer F.Cu) (net 37))
-  (segment (start 72.517 89.535) (end 72.517 91.44) (width 0.4) (layer F.Cu) (net 38))
+  (segment (start 67.437 89.789) (end 67.31 89.789) (width 0.4) (layer F.Cu) (net 37))
+  (segment (start 67.31 89.789) (end 65.659 89.789) (width 0.4) (layer F.Cu) (net 37))
+  (segment (start 72.0725 89.535) (end 72.0725 90.4875) (width 0.4) (layer F.Cu) (net 38))
+  (segment (start 72.0725 90.4875) (end 72.517 90.932) (width 0.4) (layer F.Cu) (net 38))
+  (segment (start 72.517 90.932) (end 72.517 91.44) (width 0.4) (layer F.Cu) (net 38))
+  (segment (start 72.517 91.44) (end 72.517 90.932) (width 0.4) (layer F.Cu) (net 38))
+  (segment (start 72.517 90.932) (end 72.39 90.805) (width 0.4) (layer F.Cu) (net 38))
   (segment (start 72.517 91.44) (end 74.93 91.44) (width 0.4) (layer F.Cu) (net 38))
   (segment (start 74.93 91.44) (end 75.8698 92.3798) (width 0.4) (layer F.Cu) (net 38))
